File: cad/main/main.sch (EAGLE design)
At the start: 28 parts

Commit message: schematic: add VIA, bus interface and LCD
Parts:
- added BUS_CONN: (no value), pinhead:PINHD-2X25
- added C12, C13, C14: 100nF, rcl:C-EU050-024X044
- added DIS1: TUXGR_16X2_R2, display-lcd:TUXGR_16X2_R2
- added LCD_IC: 74HC04N, 74xx-eu:74HC04N
- added LCD_POT: (no value), pot:3RP/1610N
- added R6: 3.3k, resistor:R-EU_0204/7
- added R7: 330, rcl:R-EU_0204/7
- added VIA0: W65C22S6TP, 6502:W65C22S6TP
- added VIA0_A, VIA0_B: (no value), pinhead:PINHD-1X10
- renumbered U$1 to RAM0, U$2 to RAM1, U$3 to RAM2, U$4 to RAM3
Connections:
- removed net !IO_CE: ADDR_DEC.I/O/Q09
- removed net BUS_A16: ADDR_DEC.I04, BANK_ADDR_ICA.1Q
- removed net BUS_A17: ADDR_DEC.I05, BANK_ADDR_ICA.2Q
- removed net BUS_A18: ADDR_DEC.I06, BANK_ADDR_ICA.3Q
- removed net BUS_A23: ADDR_DEC.I07, BANK_ADDR_ICA.8Q
- removed net CPU_RESB: CPU.RESB, R5.2, RESET_BTN.NO@1, RESET_BTN.NO@2
- new net !CPU_IRQ: BUS_CONN.38, CPU.IRQB, R3.1
- new net !CPU_NMIB: BUS_CONN.40, CPU.NMIB, R6.1
- new net !CPU_RESB: CPU.RESB, R5.2, RESET_BTN.NO@1, RESET_BTN.NO@2, VIA0VIA.!RESB
- new net !IO0_CE: ADDR_DEC.I/O/Q05, BUS_CONN.28, LCD_ICA.I
- new net !IO1_CE: ADDR_DEC.I/O/Q04, BUS_CONN.30, VIA0VIA.!CS2B
- new net !IO2_CE: ADDR_DEC.I/O/Q03, BUS_CONN.32
- new net !IO3_CE: ADDR_DEC.I/O/Q02, BUS_CONN.34
- new net CPU_A17: ADDR_DEC.I05, BANK_ADDR_ICA.2Q, BUS_CONN.35
- new net CPU_A18: ADDR_DEC.I06, BANK_ADDR_ICA.3Q, BUS_CONN.37
- new net CPU_A19: BANK_ADDR_ICA.4Q, BUS_CONN.39
- new net CPU_A20: BANK_ADDR_ICA.5Q, BUS_CONN.41
- new net CPU_A21: BANK_ADDR_ICA.6Q, BUS_CONN.43
- new net CPU_A22: BANK_ADDR_ICA.7Q, BUS_CONN.45
- new net CPU_A23: ADDR_DEC.I07, BANK_ADDR_ICA.8Q, BUS_CONN.47
- new net GND1: C12.2
- new net N$1: VIA0VIA.PA0, VIA0_A.1
- new net N$10: VIA0VIA.PA6, VIA0_A.7
- new net N$11: VIA0VIA.PA7, VIA0_A.8
- new net N$12: VIA0VIA.CA1, VIA0_A.9
- new net N$13: VIA0VIA.CA2, VIA0_A.10
- new net N$14: VIA0VIA.PB0, VIA0_B.1
- new net N$15: VIA0VIA.PB1, VIA0_B.2
- new net N$16: VIA0VIA.PB2, VIA0_B.3
- new net N$17: VIA0VIA.PB3, VIA0_B.4
- new net N$18: VIA0VIA.PB4, VIA0_B.5
- new net N$19: VIA0VIA.PB5, VIA0_B.6
- new net N$20: VIA0VIA.PB6, VIA0_B.7
- new net N$21: VIA0VIA.PB7, VIA0_B.8
- new net N$22: VIA0VIA.CB1, VIA0_B.9
- new net N$23: VIA0VIA.CB2, VIA0_B.10
- new net N$24: DIS1.CONTR, LCD_POT.S
- new net N$25: DIS1.E, LCD_ICA.O
- new net N$34: DIS1.NC@1, R7.2
- new net N$6: VIA0VIA.PA2, VIA0_A.3
- new net N$7: VIA0VIA.PA3, VIA0_A.4
- new net N$8: VIA0VIA.PA4, VIA0_A.5
- new net N$9: VIA0VIA.PA5, VIA0_A.6
- new net VCC1: C12.1
- net !RAM0_CE: now also ADDR_DEC.I/O/Q09; no longer ADDR_DEC.I/O/Q08, RAM1.CE1, RAM2.CE1, RAM3.CE1
- net !RAM1_CE: now also ADDR_DEC.I/O/Q08, RAM1.CE1; no longer ADDR_DEC.I/O/Q07
- net !RAM2_CE: now also ADDR_DEC.I/O/Q07, RAM2.CE1; no longer ADDR_DEC.I/O/Q06
- net !RAM3_CE: now also ADDR_DEC.I/O/Q06, RAM3.CE1; no longer ADDR_DEC.I/O/Q05
- net BUS_D0: now also BUS_CONN.4, DIS1.D0, VIA0VIA.D0
- net BUS_D1: now also BUS_CONN.6, DIS1.D1, VIA0VIA.D1
- net BUS_D2: now also BUS_CONN.8, DIS1.D2, VIA0VIA.D2
- net BUS_D3: now also BUS_CONN.10, DIS1.D3, VIA0VIA.D3
- net BUS_D4: now also BUS_CONN.12, DIS1.D4, VIA0VIA.D4
- net BUS_D5: now also BUS_CONN.14, DIS1.D5, VIA0VIA.D5
- net BUS_D6: now also BUS_CONN.16, DIS1.D6, VIA0VIA.D6
- net BUS_D7: now also BUS_CONN.18, DIS1.D7, VIA0VIA.D7
- net CLK: now also BUS_CONN.22, VIA0VIA.PHI2
- net CPU_A00: now also BUS_CONN.1, DIS1.RS, VIA0VIA.RS0
- net CPU_A01: now also BUS_CONN.3, VIA0VIA.RS1
- net CPU_A02: now also BUS_CONN.5, VIA0VIA.RS2
- net CPU_A03: now also BUS_CONN.7, VIA0VIA.RS3
- net CPU_A04: now also BUS_CONN.9
- net CPU_A05: now also BUS_CONN.11
- net CPU_A06: now also BUS_CONN.13
- net CPU_A07: now also BUS_CONN.15
- net CPU_A08: now also BUS_CONN.17
- net CPU_A09: now also BUS_CONN.19
- net CPU_A10: now also BUS_CONN.21
- net CPU_A11: now also BUS_CONN.23
- net CPU_A12: now also BUS_CONN.25
- net CPU_A13: now also BUS_CONN.27
- net CPU_A14: now also BUS_CONN.29
- net CPU_A15: now also BUS_CONN.31
- net CPU_A16: now also ADDR_DEC.I04, BANK_ADDR_ICA.1Q, BUS_CONN.33
- net CPU_RW: now also BUS_CONN.24, DIS1.R/W, VIA0VIA.R!WB
- net GND: now also BUS_CONN.20, BUS_CONN.36, BUS_CONN.49, C13.2, C14.2, DIS1.GND, DIS1.NC@2, LCD_ICP.GND, LCD_POT.E, VIA0VIAP.VSS
- net N$4: now also VIA0VIA.PA1, VIA0_A.2; no longer CPU.IRQB, R3.1
- net VCC: now also BUS_CONN.2, BUS_CONN.26, C13.1, C14.1, DIS1.VCC, LCD_ICP.VCC, LCD_POT.A, R6.2, R7.1, VIA0VIA.CS1, VIA0VIAP.VDD; no longer CPU.NMIB
Other:
- note added: "BUS Connector"
- note added: "LCD"
- note added: "VIAs"
